File: ArduPIC.kicad_pcb (KiCad board)
At the start: 2 copper layers, 50 x 50 mm, 22 parts, among them J1 PPTC141LFBN–RC, J2 PPTC121LFBN–RC, J3 3-644456-6, J4 897–43–004–90–000000, SW1 SW_SPDT, SW2 SW_DPDT_x2, SW3 1825910-6, SW4 1825910-6, U1 PIC18F2550-ISP, U2 LD1117S50TR_SOT223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

Commit message: Models update
Parts:
- PJ: renamed from PJ-002; footprint PBLE01:PJ-002 -> AditionalModels:PJ-002
- Y1: footprint PBLE01:ATS20A -> AditionalModels:ATS20A
- renumbered J4 to USB-B
Changed lines of the file:
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@@
     (property "Sheetname" "")
     (attr through_hole)
-    (fp_text reference "J4" (at 0.4815 -6.37 -90) (layer "F.SilkS")
+    (fp_text reference "USB-B" (at 0.4815 -6.37 -90) (layer "F.SilkS")
       (effects (font (size 1 1) (thickness 0.15)))
     )
@@
       (rotate (xyz 0 0 0))
     )
+    (model "${KICAD6_3DMODEL_DIR}/Button_Switch_SMD.3dshapes/SW_SPDT_PCM12.wrl"
+      (offset (xyz 0 0.2 0))
+      (scale (xyz 1.3 1.2 1.1))
+      (rotate (xyz 0 0 0))
+    )
   )
   (footprint "Capacitor_SMD:C_0805_2012Metric_Pad1.18x1.45mm_HandSolder" (layer "F.Cu")
@@
     )
   )
-  (footprint "PBLE01:ATS20A" (layer "F.Cu")
+  (footprint "AditionalModels:ATS20A" (layer "F.Cu")
     (at 136.806 67.564 180)
     (descr "ATS20A-2")
@@
     (property "Sheetname" "")
     (attr through_hole)
-    (fp_text reference "Y1" (at 2.44 0) (layer "F.SilkS")
+    (fp_text reference "Y1" (at 2.44 0 180) (layer "F.SilkS")
       (effects (font (size 1.27 1.27) (thickness 0.254)))
     )
-    (fp_text value "ATS20A" (at 2.44 0) (layer "F.SilkS") hide
+    (fp_text value "ATS20A" (at 2.44 0 180) (layer "F.SilkS") hide
       (effects (font (size 1.27 1.27) (thickness 0.254)))
     )
-    (fp_text user "${REFERENCE}" (at 2.44 0) (layer "F.Fab")
+    (fp_text user "${REFERENCE}" (at 2.44 0 180) (layer "F.Fab")
       (effects (font (size 1.27 1.27) (thickness 0.254)))
     )
-    (fp_line (start 5.615 -2.25) (end -0.735 -2.25) (layer "F.SilkS") (width 0.2))
+    (fp_line (start 5.615 2.25) (end 5.615 2.25) (layer "F.SilkS") (width 0.2))
+    (fp_line (start -0.735 -2.25) (end -0.735 -2.25) (layer "F.SilkS") (width 0.2))
+    (fp_line (start 0 2.8) (end 0 2.8) (layer "F.SilkS") (width 0.1))
     (fp_line (start -0.735 2.25) (end 5.615 2.25) (layer "F.SilkS") (width 0.2))
     (fp_line (start 0 2.9) (end 0 2.9) (layer "F.SilkS") (width 0.1))
-    (fp_line (start -0.735 -2.25) (end -0.735 -2.25) (layer "F.SilkS") (width 0.2))
-    (fp_line (start 5.615 2.25) (end 5.615 2.25) (layer "F.SilkS") (width 0.2))
-    (fp_line (start 0 2.8) (end 0 2.8) (layer "F.SilkS") (width 0.1))
+    (fp_line (start 5.615 -2.25) (end -0.735 -2.25) (layer "F.SilkS") (width 0.2))
+    (fp_arc (start -0.735 2.25) (mid -2.985 0) (end -0.735 -2.25) (layer "F.SilkS") (width 0.2))
     (fp_arc (start 0 2.8) (mid 0.05 2.85) (end 0 2.9) (layer "F.SilkS") (width 0.1))
     (fp_arc (start 0 2.9) (mid -0.05 2.85) (end 0 2.8) (layer "F.SilkS") (width 0.1))
-    (fp_arc (start -0.735 2.25) (mid -2.985 0) (end -0.735 -2.25) (layer "F.SilkS") (width 0.2))
     (fp_arc (start 5.615 -2.25) (mid 7.865 0) (end 5.615 2.25) (layer "F.SilkS") (width 0.2))
+    (fp_line (start -3.985 3.25) (end -3.985 -3.25) (layer "F.CrtYd") (width 0.1))
     (fp_line (start 8.865 3.25) (end -3.985 3.25) (layer "F.CrtYd") (width 0.1))
-    (fp_line (start -3.985 3.25) (end -3.985 -3.25) (layer "F.CrtYd") (width 0.1))
+    (fp_line (start -3.985 -3.25) (end 8.865 -3.25) (layer "F.CrtYd") (width 0.1))
     (fp_line (start 8.865 -3.25) (end 8.865 3.25) (layer "F.CrtYd") (width 0.1))
-    (fp_line (start -3.985 -3.25) (end 8.865 -3.25) (layer "F.CrtYd") (width 0.1))
+    (fp_line (start 5.615 -2.25) (end -0.735 -2.25) (layer "F.Fab") (width 0.1))
     (fp_line (start -0.735 -2.25) (end -0.735 -2.25) (layer "F.Fab") (width 0.1))
+    (fp_line (start 5.615 2.25) (end 5.615 2.25) (layer "F.Fab") (width 0.1))
     (fp_line (start -0.735 2.25) (end 5.615 2.25) (layer "F.Fab") (width 0.1))
-    (fp_line (start 5.615 2.25) (end 5.615 2.25) (layer "F.Fab") (width 0.1))
-    (fp_line (start 5.615 -2.25) (end -0.735 -2.25) (layer "F.Fab") (width 0.1))
     (fp_arc (start -0.735 2.25) (mid -2.985 0) (end -0.735 -2.25) (layer "F.Fab") (width 0.1))
     (fp_arc (start 5.615 -2.25) (mid 7.865 0) (end 5.615 2.25) (layer "F.Fab") (width 0.1))
@@
     )
   )
-  (footprint "PBLE01:PJ-002" (layer "F.Cu")
+  (footprint "AditionalModels:PJ-002" (layer "F.Cu")
     (at 115.062 93.218)
     (descr "Socket, DC power supply")
@@
     (property "Sheetname" "")
     (attr through_hole)
-    (fp_text reference "PJ-002" (at 6.858 -2.54 270) (layer "F.SilkS")
-      (effects (font (size 1 1) (thickness 0.15)))
+    (fp_text reference "PJ" (at 5.588 0.508 90) (layer "F.SilkS")
+      (effects (font (size 0.6 0.6) (thickness 0.07)))
     )
     (fp_text value "PJ-002" (at 0.11176 4.91236) (layer "F.SilkS") hide
       (effects (font (size 1.524 1.524) (thickness 0.3048)))
     )
+    (fp_line (start -4.50088 7.29996) (end 4.50088 7.29996) (layer "F.SilkS") (width 0.381))
+    (fp_line (start 4.50088 -7.29996) (end -4.50088 -7.29996) (layer "F.SilkS") (width 0.381))
+    (fp_line (start -4.50088 2.79908) (end 4.50088 2.79908) (layer "F.SilkS") (width 0.381))
+    (fp_line (start 4.50088 7.29996) (end 4.50088 -7.29996) (layer "F.SilkS") (width 0.381))
     (fp_line (start -4.50088 -7.29996) (end -4.50088 7.29996) (layer "F.SilkS") (width 0.381))
-    (fp_line (start -4.50088 2.79908) (end 4.50088 2.79908) (layer "F.SilkS") (width 0.381))
-    (fp_line (start 4.50088 -7.29996) (end -4.50088 -7.29996) (layer "F.SilkS") (width 0.381))
-    (fp_line (start -4.50088 7.29996) (end 4.50088 7.29996) (layer "F.SilkS") (width 0.381))
-    (fp_line (start 4.50088 7.29996) (end 4.50088 -7.29996) (layer "F.SilkS") (width 0.381))
     (pad "1" thru_hole oval (at 0 -6) (size 4.50088 1.99898) (drill oval 3.500119 1.00076) (layers *.Cu *.Mask "F.SilkS")
       (net 7 "Net-(CON1-Pad1)") (pintype "passive"))
