File: ArduPIC.kicad_sch (KiCad schematic)
At the start: 22 parts, among them CON1 PJ-002, SW1 SW_SPDT, SW2 SW_DPDT_x2, SW4 1825910-6, U1 PIC18F2550-ISP, U2 LD1117S50TR_SOT223

Commit message: Models update
Parts:
- C1, C3, C4: footprint (none) -> Capacitor_SMD:C_0805_2012Metric_Pad1.18x1.45mm_HandSolder
- C2, C5, C6: footprint (none) -> Capacitor_SMD:C_1206_3216Metric_Pad1.33x1.80mm_HandSolder
- CON1: value PJ-002 -> (none); footprint PBLE01:PJ-002 -> (none)
- D1: value (none) -> LTST–C150GKT; footprint (none) -> LED_SMD:LED_1206_3216Metric_Pad1.42x1.75mm_HandSolder
- J1: value (none) -> PPTC141LFBN–RC
- J2: value (none) -> PPTC121LFBN–RC
- J3: value (none) -> 3-644456-6; footprint (none) -> Connector_PinHeader_2.54mm:PinHeader_1x06_P2.54mm_Vertical
- J4: value (none) -> 897–43–004–90–000000
- R1: footprint (none) -> Resistor_SMD:R_0805_2012Metric_Pad1.20x1.40mm_HandSolder
- R2: value (none) -> 2.2k; footprint (none) -> LED_SMD:LED_0805_2012Metric_Pad1.15x1.40mm_HandSolder
- SW3: value (none) -> 1825910-6; footprint (none) -> Button_Switch_THT:SW_PUSH_6mm
- Y1: footprint (none) -> ATS20A
Changed lines of the file:
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@@
       (effects (font (size 1.27 1.27)) (justify left))
     )
-    (property "Footprint" "" (id 2) (at 68.58 57.15 0)
+    (property "Footprint" "Capacitor_SMD:C_0805_2012Metric_Pad1.18x1.45mm_HandSolder" (id 2) (at 68.58 57.15 0)
       (effects (font (size 1.27 1.27)) hide)
     )
@@
       (effects (font (size 1.27 1.27)) (justify right))
     )
-    (property "Footprint" "" (id 2) (at 68.58 137.16 0)
+    (property "Footprint" "ATS20A" (id 2) (at 68.58 137.16 0)
       (effects (font (size 1.27 1.27)) (justify left) hide)
     )
@@
       (effects (font (size 1.27 1.27)) (justify left))
     )
-    (property "Footprint" "" (id 2) (at 64.4652 173.99 0)
+    (property "Footprint" "Capacitor_SMD:C_0805_2012Metric_Pad1.18x1.45mm_HandSolder" (id 2) (at 64.4652 173.99 0)
       (effects (font (size 1.27 1.27)) hide)
     )
@@
       (effects (font (size 1.27 1.27)) hide)
     )
-    (property "Value" "" (id 1) (at 109.22 78.74 0)
+    (property "Value" "Earth" (id 1) (at 109.22 78.74 0)
       (effects (font (size 1.27 1.27)) hide)
     )
@@
       (effects (font (size 1.27 1.27)) (justify left))
     )
-    (property "Value" "" (id 1) (at 252.73 44.45 0)
+    (property "Value" "PPTC121LFBN–RC" (id 1) (at 252.73 44.45 0)
       (effects (font (size 1.27 1.27)) (justify left))
     )
@@
     (property "Reference" "C6" (id 0) (at 243.205 102.87 90))
     (property "Value" "100n" (id 1) (at 243.205 105.41 90))
-    (property "Footprint" "" (id 2) (at 243.84 110.49 0)
+    (property "Footprint" "Capacitor_SMD:C_1206_3216Metric_Pad1.33x1.80mm_HandSolder" (id 2) (at 243.84 110.49 0)
       (effects (font (size 1.27 1.27)) hide)
     )
@@
     (property "Reference" "R1" (id 0) (at 242.57 77.47 90))
     (property "Value" "10k" (id 1) (at 242.57 80.01 90))
-    (property "Footprint" "" (id 2) (at 242.57 85.598 90)
+    (property "Footprint" "Resistor_SMD:R_0805_2012Metric_Pad1.20x1.40mm_HandSolder" (id 2) (at 242.57 85.598 90)
       (effects (font (size 1.27 1.27)) hide)
     )
@@
     (in_bom yes) (on_board yes) (fields_autoplaced)
     (property "Reference" "J1" (id 0) (at 139.7 49.53 0))
-    (property "Value" "" (id 1) (at 139.7 52.07 0))
+    (property "Value" "PPTC141LFBN–RC" (id 1) (at 139.7 52.07 0))
     (property "Footprint" "Connector_PinSocket_2.54mm:PinSocket_1x14_P2.54mm_Vertical" (id 2) (at 139.7 71.12 0)
       (effects (font (size 1.27 1.27)) hide)
@@
     (in_bom yes) (on_board yes) (fields_autoplaced)
     (property "Reference" "J3" (id 0) (at 196.85 132.08 0))
-    (property "Value" "" (id 1) (at 196.85 134.62 0))
-    (property "Footprint" "" (id 2) (at 196.85 143.51 0)
+    (property "Value" "3-644456-6" (id 1) (at 196.85 134.62 0))
+    (property "Footprint" "Connector_PinHeader_2.54mm:PinHeader_1x06_P2.54mm_Vertical" (id 2) (at 196.85 143.51 0)
       (effects (font (size 1.27 1.27)) hide)
     )
@@
       (effects (font (size 1.27 1.27)) (justify right))
     )
-    (property "Value" "" (id 1) (at 113.03 71.4374 90)
+    (property "Value" "LTST–C150GKT" (id 1) (at 113.03 71.4374 90)
       (effects (font (size 1.27 1.27)) (justify right))
     )
-    (property "Footprint" "" (id 2) (at 109.22 68.58 0)
+    (property "Footprint" "LED_SMD:LED_1206_3216Metric_Pad1.42x1.75mm_HandSolder" (id 2) (at 109.22 68.58 0)
       (effects (font (size 1.27 1.27)) hide)
     )
@@
     (in_bom yes) (on_board yes) (fields_autoplaced)
     (property "Reference" "SW3" (id 0) (at 243.84 87.63 0))
-    (property "Value" "" (id 1) (at 243.84 90.17 0))
-    (property "Footprint" "" (id 2) (at 243.84 90.17 0)
+    (property "Value" "1825910-6" (id 1) (at 243.84 90.17 0))
+    (property "Footprint" "Button_Switch_THT:SW_PUSH_6mm" (id 2) (at 243.84 90.17 0)
       (effects (font (size 1.27 1.27)) hide)
     )
@@
     (in_bom yes) (on_board yes) (fields_autoplaced)
     (property "Reference" "J4" (id 0) (at 49.53 92.71 0))
-    (property "Value" "" (id 1) (at 49.53 95.25 0))
+    (property "Value" "897–43–004–90–000000" (id 1) (at 49.53 95.25 0))
     (property "Footprint" "Connector_USB:USB_B_OST_USB-B1HSxx_Horizontal" (id 2) (at 53.34 106.68 0)
       (effects (font (size 1.27 1.27)) hide)
@@
     (property "Reference" "C5" (id 0) (at 186.055 33.02 90))
     (property "Value" "100n" (id 1) (at 186.055 35.56 90))
-    (property "Footprint" "" (id 2) (at 185.42 40.64 0)
+    (property "Footprint" "Capacitor_SMD:C_1206_3216Metric_Pad1.33x1.80mm_HandSolder" (id 2) (at 185.42 40.64 0)
       (effects (font (size 1.27 1.27)) hide)
     )
@@
       (effects (font (size 1.27 1.27)) (justify left))
     )
-    (property "Footprint" "" (id 2) (at 82.2452 173.99 0)
+    (property "Footprint" "Capacitor_SMD:C_0805_2012Metric_Pad1.18x1.45mm_HandSolder" (id 2) (at 82.2452 173.99 0)
       (effects (font (size 1.27 1.27)) hide)
     )
@@
       (effects (font (size 1.524 1.524)))
     )
-    (property "Value" "PJ-002" (id 1) (at 29.8446 41.91 0)
+    (property "Value" "" (id 1) (at 29.8446 41.91 0)
       (effects (font (size 1.524 1.524)))
     )
-    (property "Footprint" "PBLE01:PJ-002" (id 2) (at 33.02 46.99 0)
+    (property "Footprint" "" (id 2) (at 33.02 46.99 0)
       (effects (font (size 1.524 1.524)) hide)
     )
@@
       (effects (font (size 1.27 1.27)) (justify left))
     )
-    (property "Footprint" "" (id 2) (at 96.52 57.15 0)
+    (property "Footprint" "Capacitor_SMD:C_1206_3216Metric_Pad1.33x1.80mm_HandSolder" (id 2) (at 96.52 57.15 0)
       (effects (font (size 1.27 1.27)) hide)
     )
@@
       (effects (font (size 1.27 1.27)) (justify left))
     )
-    (property "Value" "" (id 1) (at 111.76 58.4199 0)
-      (effects (font (size 1.27 1.27)) (justify left))
-    )
-    (property "Footprint" "" (id 2) (at 107.442 57.15 90)
+    (property "Value" "2.2k" (id 1) (at 111.76 58.4199 0)
+      (effects (font (size 1.27 1.27)) (justify left))
+    )
+    (property "Footprint" "LED_SMD:LED_0805_2012Metric_Pad1.15x1.40mm_HandSolder" (id 2) (at 107.442 57.15 90)
       (effects (font (size 1.27 1.27)) hide)
     )
@@
     )
     (path "/e65f60a3-6a43-4acf-9530-82eb35e605d5"
-      (reference "CON1") (unit 1) (value "PJ-002") (footprint "PBLE01:PJ-002")
+      (reference "CON1") (unit 1) (value "PJ-002") (footprint "AditionalModels:PJ-002")
     )
     (path "/599e717b-6f2b-4def-9eb5-8d32a29a36fa"
@@
     )
     (path "/0e847a47-b05b-4b5c-aaaf-2e9764e7bede"
-      (reference "Y1") (unit 1) (value "ATS20A") (footprint "PBLE01:ATS20A")
-    )
-  )
+      (reference "Y1") (unit 1) (value "ATS20A") (footprint "ATS20A")
+    )
+  )
